Commit message: praks 3 edasi

File: src/my_r2d2/urdf/r2d2.xacro (robot description, xacro)
@@ -216,8 +216,8 @@
     <visual>
       <geometry>
-        <cylinder radius="0.02" length="${0.02}"/>
+        <cylinder radius="0.03" length="${0.005}"/>
       </geometry>
       <material name="black"/>
-      <origin xyz="-0.04 0 0"/>
+	<origin rpy="0 1.57075 0" xyz="0 0 0"/>
     </visual>
     <collision>
@@ -231,5 +231,6 @@
     <parent link="head"/>
     <child link="lens"/>
-    <origin xyz="${.707*width+0.08} 0 ${.707*width}"/>
+    <axis xyz="0 0 1"/>
+    <origin xyz="${.707*width+0.04} 0 ${.707*width}"/>
   </joint>
 </robot>

Commit message: praks 4

File: src/my_r2d2/urdf/r2d2.xacro (robot description, xacro)
@@ -234,3 +234,11 @@
     <origin xyz="${.707*width+0.04} 0 ${.707*width}"/>
   </joint>
+  <link name="base_footprint">
+  </link>
+  <joint name="from_bf" type="fixed">
+    <parent link="base_link"/>
+    <child link="base_footprint"/>
+    <axis xyz="0 0 1"/>
+      <origin xyz="0 0 -${0.1+wheeldiam+bodylen/2}" rpy="0 0 0"/>
+  </joint>
 </robot>

Commit message: added files

File: src/my_r2d2/urdf/r2d2.xacro (robot description, xacro)
@@ -237,6 +237,6 @@
   </link>
   <joint name="from_bf" type="fixed">
-    <parent link="base_link"/>
-    <child link="base_footprint"/>
+    <parent link="base_footprint"/>
+    <child link="base_link"/>
     <axis xyz="0 0 1"/>
       <origin xyz="0 0 -${0.1+wheeldiam+bodylen/2}" rpy="0 0 0"/>

Commit message: praks5

File: src/my_r2d2/urdf/r2d2.xacro (robot description, xacro)
@@ -216,5 +216,5 @@
     <visual>
       <geometry>
-        <cylinder radius="0.03" length="${0.005}"/>
+        <cylinder radius="0.03" length="0.005"/>
       </geometry>
       <material name="black"/>
@@ -240,5 +240,12 @@
     <child link="base_link"/>
     <axis xyz="0 0 1"/>
-      <origin xyz="0 0 -${0.1+wheeldiam+bodylen/2}" rpy="0 0 0"/>
+      <origin xyz="0 0 ${0.1+wheeldiam+bodylen/2}" rpy="0 0 0"/>
+  </joint>
+  <link name="eye">
+  </link>
+  <joint name="toeye" type="continuous">
+    <parent link="lens"/>
+    <child link="eye"/>
+    <origin xyz="0 0 0" rpy="${pi} 0 0"/>
   </joint>
 </robot>

Commit message: week 30

File: src/my_r2d2/urdf/r2d2.xacro (robot description, xacro)
@@ -247,5 +247,5 @@
     <parent link="lens"/>
     <child link="eye"/>
-    <origin xyz="0 0 0" rpy="${pi} 0 0"/>
+    <origin xyz="0 0 0" rpy="${pi/2} ${pi} ${pi/2}"/>
   </joint>
 </robot>
